Commit message: intial camera logic

File: src/megajaw_description/urdf/body.xacro (robot description, xacro)
@@ -13,4 +13,9 @@
     <xacro:property name="caster_offset_x" value="${base_lx / 2 - 0.014}" />
     <xacro:property name="caster_mass" value="0.09" />
+    <xacro:property name="camera_mass" value="0.05" />
+    <xacro:property name="camera_lx" value="0.00112" />
+    <xacro:property name="camera_ly" value="0.025" />
+    <xacro:property name="camera_lz" value="0.023" />
+    <xacro:property name="camera_offset_z" value="${-base_lz / 2 + 0.04}" />
     <link name="base_footprint"></link>
     <link name="base_link">

File: src/megajaw_description/urdf/gz_plugins.xacro (robot description, xacro)
@@ -1,4 +1,5 @@
 <?xml version="1.0"?>
 <robot xmlns:xacro="http://www.ros.org/wiki/xacro">
+    <!-- ros control -->
     <gazebo>
         <plugin filename="gz_ros2_control-system" name="gz_ros2_control::GazeboSimROS2ControlPlugin">
@@ -6,3 +7,31 @@
         </plugin>
     </gazebo>
+    <!-- camera -->
+    <gazebo reference="camera_link">
+        <sensor name="camera" type="camera">
+            <camera>
+                <horizontal_fov>1.3962634</horizontal_fov>
+                <image>
+                    <width>640</width>
+                    <height>480</height>
+                    <format>R8G8B8</format>
+                </image>
+                <clip>
+                    <near>0.1</near>
+                    <far>15</far>
+                </clip>
+                <noise>
+                    <type>gaussian</type>
+                    <mean>0.0</mean>
+                    <stddev>0.007</stddev>
+                </noise>
+                <optical_frame_id>camera_link_optical</optical_frame_id>
+                <camera_info_topic>camera/camera_info</camera_info_topic>
+            </camera>
+            <always_on>1</always_on>
+            <update_rate>20</update_rate>
+            <visualize>true</visualize>
+            <topic>camera/image</topic>
+        </sensor>
+    </gazebo>
 </robot>

Commit message: working joystick

File: src/megajaw_description/urdf/body.xacro (robot description, xacro)
@@ -102,8 +102,4 @@
                 <sphere radius="${caster_radius}" />
             </geometry>
-            <friction>
-                <friction_coefficient>0.5</friction_coefficient>
-                <rolling_friction>0.1</rolling_friction>
-            </friction>
         </collision>
         <xacro:sphere_inertial m="${caster_mass}" r="${caster_radius}" o_xyz="0 0 0" o_rpy="0 0 0" />

File: src/megajaw_description/urdf/gz_plugins.xacro (robot description, xacro)
@@ -35,3 +35,29 @@
         </sensor>
     </gazebo>
+    <!-- frictions -->
+    <gazebo reference="left_wheel_link">
+        <mu1>1.0</mu1>   <!-- longitudinal friction -->
+        <mu2>1.0</mu2>   <!-- lateral friction -->
+        <fdir1>0 0 1</fdir1>  <!-- direction of mu1 (along wheel axis) -->
+        <material>Gazebo/Black</material>
+        <soft_contact>
+            <soft_cfm>0.001</soft_cfm>
+            <soft_erp>0.2</soft_erp>
+        </soft_contact>
+    </gazebo>
+    <gazebo reference="right_wheel_link">
+        <mu1>1.0</mu1>   <!-- longitudinal friction -->
+        <mu2>1.0</mu2>   <!-- lateral friction -->
+        <fdir1>0 0 1</fdir1>  <!-- direction of mu1 (along wheel axis) -->
+        <material>Gazebo/Black</material>
+        <soft_contact>
+            <soft_cfm>0.001</soft_cfm>
+            <soft_erp>0.2</soft_erp>
+        </soft_contact>
+    </gazebo>
+    <gazebo reference="caster_link">
+        <mu1>0.01</mu1>
+        <mu2>0.01</mu2>
+        <material>Gazebo/Gray</material>
+    </gazebo>
 </robot>
