Commit message: Added gripper to gazebo simulation end

File: src/megajaw_description/urdf/gz.ros2control.xacro (robot description, xacro)
@@ -18,4 +18,10 @@
             </command_interface>
         </joint>
+        <joint name="gripper_ef1_base_joint">
+            <command_interface name="position" />
+        </joint>
+        <joint name="gripper_ef2_base_joint">
+            <command_interface name="position" />
+        </joint>
     </ros2_control>
 </robot>
